File: IntelliRoastSch.sch (EAGLE design)
At the start: 28 parts, among them U1 LM2576HVS-3.3/NOPB

Commit message: Replaced Mosfet Footprint with virtical instead of horizontal
Parts:
- Q2: device transistor-power:PMOSFET_NTO220BH -> adafruit:MOSFET-NGDS_TO220V
- renumbered 12V_TERM to PWR_IN, FAN_TERM to FAN
Changed lines of the file:
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@@
 <part name="+3V2" library="supply1" library_urn="urn:adsk.eagle:library:371" deviceset="+3V3" device=""/>
 <part name="GND4" library="supply1" library_urn="urn:adsk.eagle:library:371" deviceset="GND" device=""/>
-<part name="Q2" library="transistor-power" library_urn="urn:adsk.eagle:library:400" deviceset="PMOSFET_N" device="TO220BH" package3d_urn="urn:adsk.eagle:package:29490/1"/>
+<part name="Q2" library="adafruit" library_urn="urn:adsk.eagle:library:420" deviceset="MOSFET-N" device="GDS_TO220V" package3d_urn="urn:adsk.eagle:package:6240882/1"/>
 <part name="R2" library="rcl" library_urn="urn:adsk.eagle:library:334" deviceset="R-US_" device="R0603" package3d_urn="urn:adsk.eagle:package:23555/2" value="1000"/>
-<part name="FAN_TERM" library="adafruit" deviceset="1X2" device="-3.5MM"/>
-<part name="12V_TERM" library="adafruit" deviceset="1X2" device="-3.5MM"/>
+<part name="FAN" library="adafruit" deviceset="1X2" device="-3.5MM"/>
+<part name="PWR_IN" library="adafruit" deviceset="1X2" device="-3.5MM"/>
 <part name="P+2" library="supply1" library_urn="urn:adsk.eagle:library:371" deviceset="+12V" device=""/>
 <part name="GND5" library="supply1" library_urn="urn:adsk.eagle:library:371" deviceset="GND" device=""/>
@@
 <attribute name="VALUE" x="25.4" y="50.8" size="1.778" layer="96"/>
 </instance>
-<instance part="12V_TERM" gate="G$1" x="149.86" y="71.12" smashed="yes" rot="R180"/>
+<instance part="PWR_IN" gate="G$1" x="149.86" y="71.12" smashed="yes" rot="R180"/>
 <instance part="P+2" gate="1" x="170.18" y="78.74" smashed="yes">
 <attribute name="VALUE" x="167.64" y="73.66" size="1.778" layer="96" rot="R90"/>
@@
 </segment>
 <segment>
-<pinref part="12V_TERM" gate="G$1" pin="1"/>
+<pinref part="PWR_IN" gate="G$1" pin="1"/>
 <pinref part="GND5" gate="1" pin="GND"/>
 <wire x1="154.94" y1="68.58" x2="170.18" y2="68.58" width="0.1524" layer="91"/>
@@
 </segment>
 <segment>
-<pinref part="12V_TERM" gate="G$1" pin="2"/>
+<pinref part="PWR_IN" gate="G$1" pin="2"/>
 <pinref part="P+2" gate="1" pin="+12V"/>
 <wire x1="154.94" y1="71.12" x2="170.18" y2="71.12" width="0.1524" layer="91"/>
@@
 <attribute name="VALUE" x="-4.318" y="-19.05" size="1.778" layer="96" rot="R90"/>
 </instance>
-<instance part="FAN_TERM" gate="G$1" x="-27.94" y="2.54" smashed="yes" rot="R180"/>
+<instance part="FAN" gate="G$1" x="-27.94" y="2.54" smashed="yes" rot="R180"/>
 <instance part="GND6" gate="1" x="-15.24" y="-25.4" smashed="yes">
 <attribute name="VALUE" x="-17.78" y="-27.94" size="1.778" layer="96"/>
@@
 <net name="FAN_TO_MOS" class="0">
 <segment>
-<pinref part="FAN_TERM" gate="G$1" pin="1"/>
+<pinref part="FAN" gate="G$1" pin="1"/>
 <pinref part="Q2" gate="G$1" pin="D"/>
 <wire x1="-22.86" y1="0" x2="-22.86" y2="-2.54" width="0.1524" layer="91"/>
@@
 <net name="+12V" class="0">
 <segment>
-<pinref part="FAN_TERM" gate="G$1" pin="2"/>
+<pinref part="FAN" gate="G$1" pin="2"/>
 <wire x1="-22.86" y1="2.54" x2="-22.86" y2="10.16" width="0.1524" layer="91"/>
 <pinref part="P+3" gate="1" pin="+12V"/>

Commit message: Redid the board. Should have better tolorences and the traces are better laid out. Need to add 0Ω resistors on all the connections if we need to change things around.
Parts:
- BT_HEADER: device pinhead:PINHD-1X6 -> IntelliRoast:HC-05-BREAKOUT
- TEMP0, TEMP1, TEMP2, TEMP3: device pinhead:PINHD-1X6 -> IntelliRoast:ADAFRUIT-MAX31855-BREAKOUT
- renumbered EXT_12V to EXT12V, EXT_3V3 to EXT3V3
Connections:
- net BT_ENABLE: now also CN9.15; no longer CN10.10
- net BT_STATE: now also CN9.17; no longer CN10.12
Changed lines of the file:
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@@
 <part name="P+3" library="supply1" library_urn="urn:adsk.eagle:library:371" deviceset="+12V" device=""/>
 <part name="D2" library="adafruit" library_urn="urn:adsk.eagle:library:420" deviceset="DIODE" device="SMA" package3d_urn="urn:adsk.eagle:package:6240747/1"/>
-<part name="BT_HEADER" library="pinhead" library_urn="urn:adsk.eagle:library:325" deviceset="PINHD-1X6" device="" package3d_urn="urn:adsk.eagle:package:22472/2"/>
+<part name="BT_HEADER" library="IntelliRoast" deviceset="HC-05-BREAKOUT" device=""/>
 <part name="+3V3" library="supply1" library_urn="urn:adsk.eagle:library:371" deviceset="+3V3" device=""/>
 <part name="GND7" library="supply1" library_urn="urn:adsk.eagle:library:371" deviceset="GND" device=""/>
-<part name="TEMP2" library="pinhead" library_urn="urn:adsk.eagle:library:325" deviceset="PINHD-1X6" device="" package3d_urn="urn:adsk.eagle:package:22472/2"/>
-<part name="TEMP0" library="pinhead" library_urn="urn:adsk.eagle:library:325" deviceset="PINHD-1X6" device="" package3d_urn="urn:adsk.eagle:package:22472/2"/>
-<part name="TEMP1" library="pinhead" library_urn="urn:adsk.eagle:library:325" deviceset="PINHD-1X6" device="" package3d_urn="urn:adsk.eagle:package:22472/2"/>
-<part name="TEMP3" library="pinhead" library_urn="urn:adsk.eagle:library:325" deviceset="PINHD-1X6" device="" package3d_urn="urn:adsk.eagle:package:22472/2"/>
+<part name="TEMP2" library="IntelliRoast" deviceset="ADAFRUIT-MAX31855-BREAKOUT" device=""/>
+<part name="TEMP0" library="IntelliRoast" deviceset="ADAFRUIT-MAX31855-BREAKOUT" device=""/>
+<part name="TEMP1" library="IntelliRoast" deviceset="ADAFRUIT-MAX31855-BREAKOUT" device=""/>
+<part name="TEMP3" library="IntelliRoast" deviceset="ADAFRUIT-MAX31855-BREAKOUT" device=""/>
 <part name="GND8" library="supply1" library_urn="urn:adsk.eagle:library:371" deviceset="GND" device=""/>
 <part name="GND9" library="supply1" library_urn="urn:adsk.eagle:library:371" deviceset="GND" device=""/>
@@
 <part name="GND13" library="supply1" library_urn="urn:adsk.eagle:library:371" deviceset="GND" device=""/>
 <part name="+3V9" library="supply1" library_urn="urn:adsk.eagle:library:371" deviceset="+3V3" device=""/>
-<part name="EXT_3V3" library="pinhead" library_urn="urn:adsk.eagle:library:325" deviceset="PINHD-1X2" device="" package3d_urn="urn:adsk.eagle:package:22435/2"/>
+<part name="EXT3V3" library="pinhead" library_urn="urn:adsk.eagle:library:325" deviceset="PINHD-1X2" device="" package3d_urn="urn:adsk.eagle:package:22435/2"/>
 <part name="GND14" library="supply1" library_urn="urn:adsk.eagle:library:371" deviceset="GND" device=""/>
 <part name="GND15" library="supply1" library_urn="urn:adsk.eagle:library:371" deviceset="GND" device=""/>
@@
 <part name="GND20" library="supply1" library_urn="urn:adsk.eagle:library:371" deviceset="GND" device=""/>
 <part name="P+4" library="supply1" library_urn="urn:adsk.eagle:library:371" deviceset="+12V" device=""/>
-<part name="EXT_12V" library="pinhead" library_urn="urn:adsk.eagle:library:325" deviceset="PINHD-1X2" device="" package3d_urn="urn:adsk.eagle:package:22435/2"/>
+<part name="EXT12V" library="pinhead" library_urn="urn:adsk.eagle:library:325" deviceset="PINHD-1X2" device="" package3d_urn="urn:adsk.eagle:package:22435/2"/>
 </parts>
 <sheets>
@@
 <attribute name="VALUE" x="-121.92" y="142.24" size="1.778" layer="96" rot="R90"/>
 </instance>
-<instance part="EXT_3V3" gate="G$1" x="-109.22" y="142.24" smashed="yes">
+<instance part="EXT3V3" gate="G$1" x="-109.22" y="142.24" smashed="yes">
 <attribute name="NAME" x="-115.57" y="147.955" size="1.778" layer="95"/>
 <attribute name="VALUE" x="-115.57" y="137.16" size="1.778" layer="96"/>
@@
 <attribute name="VALUE" x="-139.7" y="129.54" size="1.778" layer="96" rot="R90"/>
 </instance>
-<instance part="EXT_12V" gate="G$1" x="-129.54" y="121.92" smashed="yes">
+<instance part="EXT12V" gate="G$1" x="-129.54" y="121.92" smashed="yes">
 <attribute name="NAME" x="-135.89" y="127.635" size="1.778" layer="95"/>
 <attribute name="VALUE" x="-135.89" y="116.84" size="1.778" layer="96"/>
@@
 </segment>
 <segment>
-<pinref part="CN10" gate="G$1" pin="10"/>
-<wire x1="-25.4" y1="101.6" x2="-17.78" y2="101.6" width="0.1524" layer="91"/>
-<label x="-17.78" y="101.6" size="1.524" layer="95" xref="yes"/>
+<pinref part="CN9" gate="A" pin="15"/>
+<wire x1="-96.52" y1="96.52" x2="-104.14" y2="96.52" width="0.1524" layer="91"/>
+<label x="-104.14" y="99.06" size="1.778" layer="95" rot="R180" xref="yes"/>
+<wire x1="-104.14" y1="96.52" x2="-104.14" y2="99.06" width="0.1524" layer="91"/>
 </segment>
 </net>
@@
 </segment>
 <segment>
-<pinref part="CN10" gate="G$1" pin="12"/>
-<wire x1="-25.4" y1="99.06" x2="-17.78" y2="99.06" width="0.1524" layer="91"/>
-<label x="-17.78" y="99.06" size="1.524" layer="95" xref="yes"/>
+<pinref part="CN9" gate="A" pin="17"/>
+<wire x1="-96.52" y1="93.98" x2="-104.14" y2="93.98" width="0.1524" layer="91"/>
+<wire x1="-104.14" y1="93.98" x2="-104.14" y2="91.44" width="0.1524" layer="91"/>
+<label x="-104.14" y="91.44" size="1.778" layer="95" rot="R180" xref="yes"/>
 </segment>
 </net>
@@
 </segment>
 <segment>
-<pinref part="EXT_3V3" gate="G$1" pin="1"/>
+<pinref part="EXT3V3" gate="G$1" pin="1"/>
 <pinref part="+3V9" gate="G$1" pin="+3V3"/>
 <wire x1="-111.76" y1="144.78" x2="-119.38" y2="144.78" width="0.1524" layer="91"/>
@@
 <net name="N$2" class="0">
 <segment>
-<pinref part="EXT_3V3" gate="G$1" pin="2"/>
+<pinref part="EXT3V3" gate="G$1" pin="2"/>
 <pinref part="CN8" gate="A" pin="7"/>
 <wire x1="-111.76" y1="142.24" x2="-111.76" y2="137.16" width="0.1524" layer="91"/>
@@
 <segment>
 <pinref part="P+4" gate="1" pin="+12V"/>
-<pinref part="EXT_12V" gate="G$1" pin="1"/>
+<pinref part="EXT12V" gate="G$1" pin="1"/>
 <wire x1="-137.16" y1="132.08" x2="-137.16" y2="124.46" width="0.1524" layer="91"/>
 <wire x1="-137.16" y1="124.46" x2="-132.08" y2="124.46" width="0.1524" layer="91"/>
@@
 <net name="N$3" class="0">
 <segment>
-<pinref part="EXT_12V" gate="G$1" pin="2"/>
+<pinref part="EXT12V" gate="G$1" pin="2"/>
 <wire x1="-132.08" y1="121.92" x2="-132.08" y2="116.84" width="0.1524" layer="91"/>
 <wire x1="-132.08" y1="116.84" x2="-116.84" y2="116.84" width="0.1524" layer="91"/>
